File: Board/Controller/Drone_Controller.kicad_sch (KiCad schematic)
At the start: 6 parts, among them U1 NUCLEO144-H743ZI, U2 AT30TS74-XM8M-T, U3 ADF7020-1BCPZ, U4 BMP581, U5 VL53L1CBV0FY-1, U6 LSM6DSOTR

Commit message: I have to update the suppository
Signed-off-by: EricTheGreat <joesmith01110000011101010111@gmail.com>
Parts:
- added U7: SI4461-C2A-GMR, KiCad_Cust:IC_SI4461-C2A-GMR, symbol KiCad_Cust:SI4461-C2A-GMR
- renumbered U3 to U2, U6 to U3, U5 to U4, U4 to U5, U2 to U6
Changed lines of the file:
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@@
   (symbol (lib_id "KiCad_Cust:LSM6DSOTR") (at 191.77 62.23 0) (unit 1)
     (in_bom yes) (on_board yes)
-    (property "Reference" "U6" (id 0) (at 182.88 52.07 0))
+    (property "Reference" "U3" (id 0) (at 182.88 52.07 0))
     (property "Value" "LSM6DSOTR" (id 1) (at 191.77 72.39 0))
     (property "Footprint" "KiCad_Cust:LSM6DSOTR" (id 2) (at 179.07 54.61 0)
@@
   (symbol (lib_id "KiCad_Cust:VL53L1CBV0FY-1") (at 191.77 91.44 0) (unit 1)
     (in_bom yes) (on_board yes)
-    (property "Reference" "U5" (id 0) (at 181.61 74.93 0))
+    (property "Reference" "U4" (id 0) (at 181.61 74.93 0))
     (property "Value" "VL53L1CBV0FY-1" (id 1) (at 191.77 107.95 0))
     (property "Footprint" "KiCad_Cust:XDCR_VL53L1CBV0FY-1" (id 2) (at 191.77 91.44 0)
@@
   (symbol (lib_id "KiCad_Cust:BMP581") (at 191.77 119.38 0) (unit 1)
     (in_bom yes) (on_board yes)
-    (property "Reference" "U4" (id 0) (at 184.15 110.49 0)
+    (property "Reference" "U5" (id 0) (at 184.15 110.49 0)
       (effects (font (size 1.524 1.524)))
     )
@@
   (symbol (lib_id "KiCad_Cust:ADF7020-1BCPZ") (at 125.73 78.74 0) (unit 1)
     (in_bom yes) (on_board yes)
-    (property "Reference" "U3" (id 0) (at 111.76 16.51 0))
+    (property "Reference" "U2" (id 0) (at 111.76 16.51 0))
     (property "Value" "ADF7020-1BCPZ" (id 1) (at 125.73 78.74 0))
     (property "Footprint" "Package_DFN_QFN:VQFN-48-1EP_7x7mm_P0.5mm_EP5.15x5.15mm_ThermalVias" (id 2) (at 125.73 78.74 0)
@@
     (pin "9")
   )
+  (symbol (lib_id "KiCad_Cust:SI4461-C2A-GMR") (at 191.77 184.15 0) (unit 1)
+    (in_bom yes) (on_board yes) (fields_autoplaced)
+    (property "Reference" "U7" (id 0) (at 191.77 156.21 0))
+    (property "Value" "SI4461-C2A-GMR" (id 1) (at 191.77 158.75 0))
+    (property "Footprint" "KiCad_Cust:IC_SI4461-C2A-GMR" (id 2) (at 191.77 184.15 0)
+      (effects (font (size 1.27 1.27)) (justify left bottom) hide)
+    )
+    (property "Datasheet" "" (id 3) (at 191.77 184.15 0)
+      (effects (font (size 1.27 1.27)) (justify left bottom) hide)
+    )
+    (property "DigiKey-Purchase-URL" "https://snapeda.com/shop?store=DigiKey&id=588592" (id 4) (at 191.77 184.15 0)
+      (effects (font (size 1.27 1.27)) (justify left bottom) hide)
+    )
+    (property "Availability" "Unavailable" (id 5) (at 191.77 184.15 0)
+      (effects (font (size 1.27 1.27)) (justify left bottom) hide)
+    )
+    (property "MP" "SI4461-C2A-GMR" (id 6) (at 191.77 184.15 0)
+      (effects (font (size 1.27 1.27)) (justify left bottom) hide)
+    )
+    (property "MF" "Silicon Labs" (id 7) (at 191.77 184.15 0)
+      (effects (font (size 1.27 1.27)) (justify left bottom) hide)
+    )
+    (property "Package" "QFN-20 Silicon Labs" (id 8) (at 191.77 184.15 0)
+      (effects (font (size 1.27 1.27)) (justify left bottom) hide)
+    )
+    (property "Description" "IC RF TxRx + MCU General ISM < 1GHz 142MHz ~{} 1.05GHz 20-VFQFN Exposed Pad" (id 9) (at 191.77 184.15 0)
+      (effects (font (size 1.27 1.27)) (justify left bottom) hide)
+    )
+    (property "Price" "None" (id 10) (at 191.77 184.15 0)
+      (effects (font (size 1.27 1.27)) (justify left bottom) hide)
+    )
+    (pin "1")
+    (pin "10")
+    (pin "11")
+    (pin "12")
+    (pin "13")
+    (pin "14")
+    (pin "15")
+    (pin "16")
+    (pin "17")
+    (pin "18")
+    (pin "19")
+    (pin "2")
+    (pin "20")
+    (pin "21")
+    (pin "3")
+    (pin "4")
+    (pin "5")
+    (pin "6")
+    (pin "7")
+    (pin "8")
+    (pin "9")
+  )
   (symbol (lib_id "KiCad_Cust:AT30TS74-XM8M-T") (at 191.77 137.16 0) (unit 1)
     (in_bom yes) (on_board yes)
-    (property "Reference" "U2" (id 0) (at 186.69 130.81 0))
+    (property "Reference" "U6" (id 0) (at 186.69 130.81 0))
     (property "Value" "AT30TS74-XM8M-T" (id 1) (at 191.77 143.51 0))
     (property "Footprint" "Package_SO:MSOP-8_3x3mm_P0.65mm" (id 2) (at 191.77 137.16 0)
@@
       (reference "U1") (unit 1) (value "NUCLEO144-H743ZI") (footprint "Module:ST_Morpho_Connector_144_STLink")
     )
+    (path "/a8378168-7ba9-4a66-baf2-4fc237ddf333"
+      (reference "U2") (unit 1) (value "ADF7020-1BCPZ") (footprint "Package_DFN_QFN:VQFN-48-1EP_7x7mm_P0.5mm_EP5.15x5.15mm_ThermalVias")
+    )
+    (path "/52e12011-0a99-4e20-9e0d-d0405fcfff1e"
+      (reference "U3") (unit 1) (value "LSM6DSOTR") (footprint "KiCad_Cust:LSM6DSOTR")
+    )
+    (path "/857e1a05-bc14-4a54-b833-3e1c74aeae61"
+      (reference "U4") (unit 1) (value "VL53L1CBV0FY-1") (footprint "KiCad_Cust:XDCR_VL53L1CBV0FY-1")
+    )
+    (path "/9181bd00-098e-4db9-8ae0-e3a266f35a69"
+      (reference "U5") (unit 1) (value "BMP581") (footprint "KiCad_Cust:BMP581")
+    )
     (path "/ceb25cf7-d36f-4f0e-bf85-8b967964b0f3"
-      (reference "U2") (unit 1) (value "AT30TS74-XM8M-T") (footprint "Package_SO:MSOP-8_3x3mm_P0.65mm")
-    )
-    (path "/a8378168-7ba9-4a66-baf2-4fc237ddf333"
-      (reference "U3") (unit 1) (value "ADF7020-1BCPZ") (footprint "Package_DFN_QFN:VQFN-48-1EP_7x7mm_P0.5mm_EP5.15x5.15mm_ThermalVias")
-    )
-    (path "/9181bd00-098e-4db9-8ae0-e3a266f35a69"
-      (reference "U4") (unit 1) (value "BMP581") (footprint "KiCad_Cust:BMP581")
-    )
-    (path "/857e1a05-bc14-4a54-b833-3e1c74aeae61"
-      (reference "U5") (unit 1) (value "VL53L1CBV0FY-1") (footprint "KiCad_Cust:XDCR_VL53L1CBV0FY-1")
-    )
-    (path "/52e12011-0a99-4e20-9e0d-d0405fcfff1e"
-      (reference "U6") (unit 1) (value "LSM6DSOTR") (footprint "KiCad_Cust:LSM6DSOTR")
-    )
-  )
+      (reference "U6") (unit 1) (value "AT30TS74-XM8M-T") (footprint "Package_SO:MSOP-8_3x3mm_P0.65mm")
+    )
+    (path "/c195be24-c988-452d-b72d-6611cbe671f7"
+      (reference "U7") (unit 1) (value "SI4461-C2A-GMR") (footprint "KiCad_Cust:IC_SI4461-C2A-GMR")
+    )
+  )

Commit message: we did stuff
Signed-off-by: EricTheGreat <joesmith01110000011101010111@gmail.com>
Parts:
- removed U2: ADF7020-1BCPZ, Package_DFN_QFN:VQFN-48-1EP_7x7mm_P0.5mm_EP5.15x5.15mm_ThermalVias, symbol KiCad_Cust:ADF7020-1BCPZ
- removed U7: SI4461-C2A-GMR, KiCad_Cust:IC_SI4461-C2A-GMR, symbol KiCad_Cust:SI4461-C2A-GMR
- added C1, C2: .1uF, Resistor_SMD:R_0805_2012Metric, symbol Device:C_Small
- renumbered U5 to U2, U4 to U3, U6 to U4, U3 to U5
Connections:
- net +3V3: now reaches U2.1 (VDDIO)
- net +3V3: now also U2.10 (VDD), C1.1, C2.1
- net SPI1_SCK: now reaches U2.2 (SCK)
- net SPI1_SCK: now also U1.83 (PA5)
- net GND: now reaches U2.3 (VSS)
- net GND: now also U2.8 (VSS), U2.9 (VSS), C1.2, C2.2
- net SPI1_MOSI: now reaches U2.4 (SDI)
- net SPI1_MOSI: now also U1.45 (PD7)
- net SPI1_MISO: now reaches U2.5 (SDO)
- net SPI1_MISO: now also U1.85 (PA6)
- net SPI1_NSS: now reaches U2.6 (CSB)
- net SPI1_NSS: now also U1.32 (PA4)
- net BMP_INT: now reaches U2.7 (INT)
Other:
- moved on the sheet: U2, U3, U4, U5

Commit message: yo
Signed-off-by: EricTheGreat <joesmith01110000011101010111@gmail.com>
Parts:
- added C? (x3): .1uF, Resistor_SMD:R_0805_2012Metric, symbol Device:C_Small
- added R?: 2k, Resistor_SMD:R_0805_2012Metric, symbol Device:R_Small_US
Connections:
- net +3V3: now also U3.1 (AVDDVCSEL), U3.11 (AVDD), U5.5 (VDDIO), U5.8 (VDD), C?.1, C?.1, C?.1
- net GND: now also U3.12 (GND4), U3.2 (AVSSVCSEL), U3.3 (GND), U3.4 (GND2), U3.6 (GND3), U5.6 (GND), U5.7 (GND), C?.2, C?.2, C?.2, R?.2
- net SPI2_MISO: now reaches U5.1 (SDO/SA0)
- net SPI2_NSS: now reaches U5.12 (CS)
- net SPI2_SCK: now reaches U5.13 (SCL)
- net SPI2_MOSI: now reaches U5.14 (SDA)
- net IMU_EXT: now reaches U5.4 (INT1)
- net at U3.5 (~{XSHUT}): now also R?.1
- net BMP_INT renamed BMP_EXT
Other:
- moved on the sheet: U3, U5

Commit message: tt
Parts:
- added R? (x3): 2k, Resistor_SMD:R_0805_2012Metric, symbol Device:R_Small_US
Connections:
- net +3V3: now also R?.1, R?.1, R?.1
- net at U3.10 (SCL): now also R?.2
- net at U3.7 (GPIO1): now also R?.2
- net at U3.9 (SDA): now also R?.2
Changed lines of the file:
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@@
+    (stroke (width 0) (type default) (color 0 0 0 0))
+  )
+  (wire (pts (xy 173.99 148.59) (xy 173.99 160.02))
+    (stroke (width 0) (type default) (color 0 0 0 0))
+  )
+  (wire (pts (xy 173.99 160.02) (xy 193.04 160.02))
     (stroke (width 0) (type default) (color 0 0 0 0))
   )
@@
     (stroke (width 0) (type default) (color 0 0 0 0))
   )
+  (wire (pts (xy 180.34 140.97) (xy 180.34 143.51))
+    (stroke (width 0) (type default) (color 0 0 0 0))
+  )
   (wire (pts (xy 182.88 46.99) (xy 182.88 59.69))
     (stroke (width 0) (type default) (color 0 0 0 0))
@@
     (stroke (width 0) (type default) (color 0 0 0 0))
   )
+  (wire (pts (xy 173.99 140.97) (xy 173.99 143.51))
+    (stroke (width 0) (type default) (color 0 0 0 0))
+  )
   (wire (pts (xy 86.36 46.99) (xy 88.9 46.99))
     (stroke (width 0) (type default) (color 0 0 0 0))
@@
     (stroke (width 0) (type default) (color 0 0 0 0))
   )
+  (wire (pts (xy 180.34 148.59) (xy 180.34 157.48))
+    (stroke (width 0) (type default) (color 0 0 0 0))
+  )
   (wire (pts (xy 223.52 111.76) (xy 232.41 111.76))
     (stroke (width 0) (type default) (color 0 0 0 0))
   )
+  (wire (pts (xy 186.69 140.97) (xy 186.69 143.51))
+    (stroke (width 0) (type default) (color 0 0 0 0))
+  )
   (wire (pts (xy 86.36 52.07) (xy 88.9 52.07))
     (stroke (width 0) (type default) (color 0 0 0 0))
@@
     (stroke (width 0) (type default) (color 0 0 0 0))
   )
+  (wire (pts (xy 186.69 148.59) (xy 186.69 152.4))
+    (stroke (width 0) (type default) (color 0 0 0 0))
+  )
   (wire (pts (xy 229.87 165.1) (xy 229.87 162.56))
     (stroke (width 0) (type default) (color 0 0 0 0))
@@
     (stroke (width 0) (type default) (color 0 0 0 0))
   )
+  (wire (pts (xy 180.34 157.48) (xy 193.04 157.48))
+    (stroke (width 0) (type default) (color 0 0 0 0))
+  )
   (wire (pts (xy 140.97 52.07) (xy 142.24 52.07))
     (stroke (width 0) (type default) (color 0 0 0 0))
@@
   )
   (wire (pts (xy 228.6 162.56) (xy 229.87 162.56))
+    (stroke (width 0) (type default) (color 0 0 0 0))
+  )
+  (wire (pts (xy 186.69 152.4) (xy 193.04 152.4))
     (stroke (width 0) (type default) (color 0 0 0 0))
   )
@@
     (pin "2")
   )
+  (symbol (lib_id "Device:R_Small_US") (at 186.69 146.05 0) (unit 1)
+    (in_bom yes) (on_board yes) (fields_autoplaced)
+    (property "Reference" "R?" (id 0) (at 189.23 144.7799 0)
+      (effects (font (size 1.27 1.27)) (justify left))
+    )
+    (property "Value" "2k" (id 1) (at 189.23 147.3199 0)
+      (effects (font (size 1.27 1.27)) (justify left))
+    )
+    (property "Footprint" "Resistor_SMD:R_0805_2012Metric" (id 2) (at 186.69 146.05 0)
+      (effects (font (size 1.27 1.27)) hide)
+    )
+    (property "Datasheet" "~" (id 3) (at 186.69 146.05 0)
+      (effects (font (size 1.27 1.27)) hide)
+    )
+    (pin "1")
+    (pin "2")
+  )
   (symbol (lib_id "Device:R_Small_US") (at 191.77 165.1 0) (unit 1)
     (in_bom yes) (on_board yes) (fields_autoplaced)
@@
     )
     (property "Datasheet" "~" (id 3) (at 191.77 165.1 0)
+      (effects (font (size 1.27 1.27)) hide)
+    )
+    (pin "1")
+    (pin "2")
+  )
+  (symbol (lib_id "Device:R_Small_US") (at 180.34 146.05 0) (unit 1)
+    (in_bom yes) (on_board yes) (fields_autoplaced)
+    (property "Reference" "R?" (id 0) (at 182.88 144.7799 0)
+      (effects (font (size 1.27 1.27)) (justify left))
+    )
+    (property "Value" "2k" (id 1) (at 182.88 147.3199 0)
+      (effects (font (size 1.27 1.27)) (justify left))
+    )
+    (property "Footprint" "Resistor_SMD:R_0805_2012Metric" (id 2) (at 180.34 146.05 0)
+      (effects (font (size 1.27 1.27)) hide)
+    )
+    (property "Datasheet" "~" (id 3) (at 180.34 146.05 0)
       (effects (font (size 1.27 1.27)) hide)
     )
@@
     )
     (property "Datasheet" "" (id 3) (at 229.87 170.18 0)
+      (effects (font (size 1.27 1.27)) hide)
+    )
+    (pin "1")
+  )
+  (symbol (lib_id "power:+3.3V") (at 173.99 140.97 0) (unit 1)
+    (in_bom yes) (on_board yes)
+    (property "Reference" "#PWR?" (id 0) (at 173.99 144.78 0)
+      (effects (font (size 1.27 1.27)) hide)
+    )
+    (property "Value" "+3.3V" (id 1) (at 173.99 137.16 0))
+    (property "Footprint" "" (id 2) (at 173.99 140.97 0)
+      (effects (font (size 1.27 1.27)) hide)
+    )
+    (property "Datasheet" "" (id 3) (at 173.99 140.97 0)
       (effects (font (size 1.27 1.27)) hide)
     )
@@
     (pin "8")
     (pin "9")
+  )
+  (symbol (lib_id "power:+3.3V") (at 186.69 140.97 0) (unit 1)
+    (in_bom yes) (on_board yes)
+    (property "Reference" "#PWR?" (id 0) (at 186.69 144.78 0)
+      (effects (font (size 1.27 1.27)) hide)
+    )
+    (property "Value" "+3.3V" (id 1) (at 186.69 137.16 0))
+    (property "Footprint" "" (id 2) (at 186.69 140.97 0)
+      (effects (font (size 1.27 1.27)) hide)
+    )
+    (property "Datasheet" "" (id 3) (at 186.69 140.97 0)
+      (effects (font (size 1.27 1.27)) hide)
+    )
+    (pin "1")
   )
   (symbol (lib_id "power:GND") (at 140.97 66.04 0) (unit 1)
@@
     (pin "99")
   )
+  (symbol (lib_id "power:+3.3V") (at 180.34 140.97 0) (unit 1)
+    (in_bom yes) (on_board yes)
+    (property "Reference" "#PWR?" (id 0) (at 180.34 144.78 0)
+      (effects (font (size 1.27 1.27)) hide)
+    )
+    (property "Value" "+3.3V" (id 1) (at 180.34 137.16 0))
+    (property "Footprint" "" (id 2) (at 180.34 140.97 0)
+      (effects (font (size 1.27 1.27)) hide)
+    )
+    (property "Datasheet" "" (id 3) (at 180.34 140.97 0)
+      (effects (font (size 1.27 1.27)) hide)
+    )
+    (pin "1")
+  )
   (symbol (lib_id "power:+3.3V") (at 226.06 97.79 0) (unit 1)
     (in_bom yes) (on_board yes)
@@
     )
     (pin "1")
+  )
+  (symbol (lib_id "Device:R_Small_US") (at 173.99 146.05 0) (unit 1)
+    (in_bom yes) (on_board yes) (fields_autoplaced)
+    (property "Reference" "R?" (id 0) (at 176.53 144.7799 0)
+      (effects (font (size 1.27 1.27)) (justify left))
+    )
+    (property "Value" "2k" (id 1) (at 176.53 147.3199 0)
+      (effects (font (size 1.27 1.27)) (justify left))
+    )
+    (property "Footprint" "Resistor_SMD:R_0805_2012Metric" (id 2) (at 173.99 146.05 0)
+      (effects (font (size 1.27 1.27)) hide)
+    )
+    (property "Datasheet" "~" (id 3) (at 173.99 146.05 0)
+      (effects (font (size 1.27 1.27)) hide)
+    )
+    (pin "1")
+    (pin "2")
   )
   (sheet_instances
@@
       (reference "#PWR?") (unit 1) (value "GND") (footprint "")
     )
+    (path "/480725f4-a74b-4123-930b-e7269f522bc3"
+      (reference "#PWR?") (unit 1) (value "+3.3V") (footprint "")
+    )
     (path "/4e975022-511a-4407-8dc1-5c9bf677ac07"
       (reference "#PWR?") (unit 1) (value "GND") (footprint "")
@@
       (reference "#PWR?") (unit 1) (value "GND") (footprint "")
     )
+    (path "/98bdd80a-ad36-40dc-a10c-f3f85578e90b"
+      (reference "#PWR?") (unit 1) (value "+3.3V") (footprint "")
+    )
     (path "/bdb52708-752f-43ad-b9d1-155aade5b868"
       (reference "#PWR?") (unit 1) (value "GND") (footprint "")
     )
+    (path "/dc419653-30d5-4e3e-9562-e0e5d53120a6"
+      (reference "#PWR?") (unit 1) (value "+3.3V") (footprint "")
+    )
     (path "/df26e74b-d3e8-42be-a468-53fe16f8ab6b"
       (reference "#PWR?") (unit 1) (value "+3.3V") (footprint "")
@@
       (reference "C?") (unit 1) (value ".1uF") (footprint "Resistor_SMD:R_0805_2012Metric")
     )
+    (path "/2f4187ae-7293-4d82-b476-5281f2da45bd"
+      (reference "R?") (unit 1) (value "2k") (footprint "Resistor_SMD:R_0805_2012Metric")
+    )
     (path "/31dd03fa-f91d-4e4d-a492-4ce6baabc3e5"
       (reference "R?") (unit 1) (value "2k") (footprint "Resistor_SMD:R_0805_2012Metric")
     )
+    (path "/3464444c-628f-48de-8708-5f1df8cf2a8b"
+      (reference "R?") (unit 1) (value "2k") (footprint "Resistor_SMD:R_0805_2012Metric")
+    )
+    (path "/f36feab9-335e-45f0-b054-7d64353766dd"
+      (reference "R?") (unit 1) (value "2k") (footprint "Resistor_SMD:R_0805_2012Metric")
+    )
